File: Battery Charger Project/KiCad/Build/_autosave-Build.kicad_sch (KiCad schematic)
At the start: 21 parts, among them J1 Screw_Terminal_01x03, J2 Screw_Terminal_01x03, J3 Screw_Terminal_01x02, J5 726386-2, J6 726386-2, J9 726386-2, U1 LAUNCHXL-F28379D, U2 TMCS1133C3A

Commit message: Save push
Connections:
- net +3.3V renamed +5V
Changed lines of the file:
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@@
 			)
 		)
-		(property "Value" "+3.3V"
+		(property "Value" "+5V"
 			(at 207.01 28.702 90)
 			(show_name no)
