File: Battery Charger Project/KiCad/Build/Build.kicad_pcb (KiCad board)
At the start: 2 copper layers, 135 x 119.2 mm, 26 parts, among them J1 Screw_Terminal_01x03, J2 Screw_Terminal_01x02, J3 Screw_Terminal_01x03, J4 726386-2, J5 726386-2, J6 726386-2, U1 LAUNCHXL-F28379D, U2 TMCS1133C3A

Commit message: PCB updates
Added larger planes and a top ground pour connected to the rec to help with the bottleneck. Also put some vias to distribute current and heat
Routing:
- net Net-(U2-IN+): vias 0 -> 4
- net GND: vias 4 -> 16
Changed lines of the file:
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@@
 			)
 		)
-		(property "Datasheet" "https://ixapps.ixys.com/Datasheet/DNA40U2200GU.pdf"
+		(property "Datasheet" ""
 			(at 0 0 180)
 			(unlocked yes)
@@
 			)
 		)
-		(property "Description" "690V Vrms, 40A If, GUFP(X025B)"
+		(property "Description" ""
 			(at 0 0 180)
 			(unlocked yes)
@@
 		(sheetname "/")
 		(sheetfile "Build.kicad_sch")
-		(units
-			(unit
-				(name "A")
-				(pins "5" "4" "3" "1" "2")
-			)
-		)
 		(attr through_hole)
 		(duplicate_pad_numbers_are_jumpers no)
@@
 		(pad "1" thru_hole roundrect
 			(at 0 7.747 180)
-			(size 2 2.4)
+			(size 2 2.2)
 			(drill oval 0.9 1.6)
 			(layers "*.Cu" "*.Mask")
@@
 		(pad "2" thru_hole roundrect
 			(at 0 3.937 180)
-			(size 2 2.4)
+			(size 2 2.2)
 			(drill oval 0.9 1.6)
 			(layers "*.Cu" "*.Mask")
@@
 		(pad "3" thru_hole roundrect
 			(at 0 0.127 180)
-			(size 2 2.4)
+			(size 2 2.2)
 			(drill oval 0.9 1.6)
 			(layers "*.Cu" "*.Mask")
@@
 		(pad "4" thru_hole roundrect
 			(at 0 -3.683 180)
-			(size 2 2.4)
+			(size 2 2.2)
 			(drill oval 0.9 1.6)
 			(layers "*.Cu" "*.Mask")
@@
 		(pad "5" thru_hole roundrect
 			(at 0 -7.493 180)
-			(size 2 2.4)
+			(size 2 2.2)
 			(drill oval 0.9 1.6)
 			(layers "*.Cu" "*.Mask")
@@
 	)
 	(via
+		(at 103.03 133.46)
+		(size 0.6)
+		(drill 0.4)
+		(layers "F.Cu" "B.Cu")
+		(free yes)
+		(net "GND")
+	)
+	(via
 		(at 135.9 81)
 		(size 0.6)
@@
 	)
 	(via
+		(at 91.71 126.28)
+		(size 0.6)
+		(drill 0.4)
+		(layers "F.Cu" "B.Cu")
+		(free yes)
+		(net "GND")
+	)
+	(via
+		(at 96.11 126.28)
+		(size 0.6)
+		(drill 0.4)
+		(layers "F.Cu" "B.Cu")
+		(free yes)
+		(net "GND")
+	)
+	(via
+		(at 93.91 126.28)
+		(size 0.6)
+		(drill 0.4)
+		(layers "F.Cu" "B.Cu")
+		(free yes)
+		(net "GND")
+	)
+	(via
+		(at 92.91 124.78)
+		(size 0.6)
+		(drill 0.4)
+		(layers "F.Cu" "B.Cu")
+		(free yes)
+		(net "GND")
+	)
+	(via
+		(at 103.03 131.66)
+		(size 0.6)
+		(drill 0.4)
+		(layers "F.Cu" "B.Cu")
+		(free yes)
+		(net "GND")
+	)
+	(via
+		(at 90.71 124.78)
+		(size 0.6)
+		(drill 0.4)
+		(layers "F.Cu" "B.Cu")
+		(free yes)
+		(net "GND")
+	)
+	(via
 		(at 129.85 90.15)
 		(size 0.6)
@@
 	)
 	(via
+		(at 95.11 124.78)
+		(size 0.6)
+		(drill 0.4)
+		(layers "F.Cu" "B.Cu")
+		(free yes)
+		(net "GND")
+	)
+	(via
+		(at 104.53 134.36)
+		(size 0.6)
+		(drill 0.4)
+		(layers "F.Cu" "B.Cu")
+		(free yes)
+		(net "GND")
+	)
+	(via
 		(at 117.6 74)
 		(size 0.6)
@@
 		(net "GND")
 	)
+	(via
+		(at 104.53 130.76)
+		(size 0.6)
+		(drill 0.4)
+		(layers "F.Cu" "B.Cu")
+		(free yes)
+		(net "GND")
+	)
+	(via
+		(at 104.53 132.56)
+		(size 0.6)
+		(drill 0.4)
+		(layers "F.Cu" "B.Cu")
+		(free yes)
+		(net "GND")
+	)
+	(via
+		(at 103.03 129.86)
+		(size 0.6)
+		(drill 0.4)
+		(layers "F.Cu" "B.Cu")
+		(free yes)
+		(net "GND")
+	)
 	(segment
 		(start 130.275 89.725)
@@
 		(net "5V")
 	)
+	(via
+		(at 151.43 94.52)
+		(size 0.6)
+		(drill 0.4)
+		(layers "F.Cu" "B.Cu")
+		(free yes)
+		(net "Net-(U2-IN+)")
+	)
+	(via
+		(at 151.43 96.52)
+		(size 0.6)
+		(drill 0.4)
+		(layers "F.Cu" "B.Cu")
+		(free yes)
+		(net "Net-(U2-IN+)")
+	)
+	(via
+		(at 153.43 96.52)
+		(size 0.6)
+		(drill 0.4)
+		(layers "F.Cu" "B.Cu")
+		(free yes)
+		(net "Net-(U2-IN+)")
+	)
+	(via
+		(at 153.43 94.52)
+		(size 0.6)
+		(drill 0.4)
+		(layers "F.Cu" "B.Cu")
+		(free yes)
+		(net "Net-(U2-IN+)")
+	)
 	(segment
 		(start 184.3625 36.7375)
@@
 		(polygon
 			(pts
+				(xy 112.25 129.1) (xy 112.3 135.2) (xy 103.5 135.2) (xy 101.9 133.6) (xy 96.7 133.65) (xy 94.2 130.75)
+				(xy 85 119.65) (xy 85 114.6) (xy 92.9 114.6) (xy 92.9 120.825269) (xy 97.55 125.425269) (xy 97.55 129.1)
+				(xy 98.25 129.1)
+			)
+		)
+	)
+	(zone
+		(net "GND")
+		(layer "F.Cu")
+		(hatch edge 0.5)
+		(connect_pads yes
+			(clearance 0.5)
+		)
+		(min_thickness 0.25)
+		(fill yes
+			(thermal_gap 0.5)
+			(thermal_bridge_width 0.5)
+			(island_removal_mode 1)
+		)
+		(polygon
+			(pts
 				(xy 216 28) (xy 86.1 28) (xy 86.066694 82) (xy 216 81.9)
 			)
@@
 		(polygon
 			(pts
-				(xy 85 119.7) (xy 85 110) (xy 105.15 110) (xy 112.25 102.8) (xy 140.4 102.8) (xy 149.1 111.5) (xy 149.1 135.2)
-				(xy 104.5 135.2) (xy 104.5 128.4) (xy 93.7 128.4)
+				(xy 113.780621 138.62) (xy 149.090702 138.62) (xy 149.090702 111.575) (xy 140.390702 102.875) (xy 112.240702 102.875)
+				(xy 105.633759 109.575) (xy 105.588409 109.625) (xy 100.835 109.625) (xy 98.05 106.84) (xy 84.990702 106.84)
+				(xy 84.990702 113.199999) (xy 94.240702 113.249999) (xy 94.240702 120.25) (xy 98.415702 124.425)
+				(xy 98.415702 128.2) (xy 100.46 128.21) (xy 100.885 127.81) (xy 113.779674 127.81)
 			)
 		)
 	)
 	(zone
-		(net "/C")
+		(net "/B")
 		(layers "F.Cu" "B.Cu")
 		(hatch edge 0.5)
-		(priority 2)
 		(connect_pads yes
 			(clearance 0.5)
@@
 		(polygon
 			(pts
-				(xy 100.8 143.820358) (xy 97.9 143.820358) (xy 88.8 143.220358) (xy 88.7 140.220358) (xy 97.1 140.920358)
-				(xy 100.8 140.920358)
+				(xy 88.37 139.61) (xy 91.5 139.61) (xy 92.3 140.41) (xy 96.46 140.41) (xy 100.51 140.41) (xy 100.51 136.93)
+				(xy 91.795474 136.93) (xy 90.855474 135.98) (xy 88.37 135.98) (xy 88.37 139.03)
 			)
 		)
 	)
 	(zone
-		(net "/A")
+		(net "/C")
 		(layers "F.Cu" "B.Cu")
 		(hatch edge 0.5)
@@
 		(polygon
 			(pts
-				(xy 88.564661 130.136222) (xy 88.6 133.115707) (xy 97.213333 136.120358) (xy 100.7 136.120358) (xy 100.735175 133.520221)
-				(xy 98.004224 133.530984)
+				(xy 88.89 144.63) (xy 100.48 144.64) (xy 100.48 141.28) (xy 91.52 141.297659) (xy 91.52 140.7) (xy 88.89 140.702181)
 			)
 		)
 	)
 	(zone
-		(net "Net-(U2-IN+)")
+		(net "/A")
 		(layers "F.Cu" "B.Cu")
 		(hatch edge 0.5)
+		(priority 2)
 		(connect_pads yes
 			(clearance 0.5)
@@
 		(polygon
 			(pts
-				(xy 179.2 93.7) (xy 150.6 93.7) (xy 150.6 98.8) (xy 170.7 98.8) (xy 170.7 100.1) (xy 179.2 100.1)
+				(xy 88.564661 130.136222) (xy 88.53 134.32) (xy 98.61 135.82) (xy 100.485119 135.8) (xy 100.514935 133.595998)
+				(xy 98.210263 133.605082)
 			)
 		)
 	)
 	(zone
-		(net "/B")
+		(net "Net-(U2-IN+)")
 		(layers "F.Cu" "B.Cu")
 		(hatch edge 0.5)
-		(priority 1)
+		(priority 4)
 		(connect_pads yes
 			(clearance 0.5)
@@
 		(polygon
 			(pts
-				(xy 88.8 138.26675) (xy 96.5 139.920358) (xy 100.7 139.920358) (xy 100.7 137.120358) (xy 97.1 137.120358)
-				(xy 88.8 135.320358)
+				(xy 179.2 93.7) (xy 150.6 93.7) (xy 150.6 98.8) (xy 170.7 98.8) (xy 170.7 100.1) (xy 179.2 100.1)
 			)
 		)
@@
 		(layers "F.Cu" "B.Cu")
 		(hatch edge 0.5)
+		(priority 6)
 		(connect_pads yes
 			(clearance 0.5)
@@
 		(layer "B.Cu")
 		(hatch edge 0.5)
+		(priority 1)
 		(connect_pads yes
 			(clearance 0.5)
@@
 		(polygon
 			(pts
-				(xy 152.8 104.6) (xy 141.6 115.8) (xy 141.6 135.2) (xy 104.5 135.2) (xy 104.5 132.2) (xy 97.6 132.2)
-				(xy 85 119.6) (xy 85 102.883399) (xy 130 102.8) (xy 131.9 102.8) (xy 135.3 99.4) (xy 152.8 99.4)
+				(xy 152.8 104.6) (xy 141.6 115.8) (xy 141.6 135.2) (xy 104.5 135.2) (xy 103.5 135.2) (xy 101.92 133.65)
+				(xy 96.7 133.65) (xy 85 119.65) (xy 85 102.883399) (xy 130 102.8) (xy 131.9 102.8) (xy 135.3 99.4)
+				(xy 152.8 99.4)
 			)
 		)
@@
 		(layer "B.Cu")
 		(hatch edge 0.5)
+		(priority 5)
 		(connect_pads yes
 			(clearance 0.5)
@@
 		(layer "B.Cu")
 		(hatch edge 0.5)
+		(priority 7)
 		(connect_pads yes
 			(clearance 0.5)

Commit message: PCB updates
Parts:
- added C11: C_Small, Capacitor_SMD:C_0805_2012Metric_Pad1.18x1.45mm_HandSolder, B.Cu at (149.2, 86.0)
- moved C4 20.1 mm to (159.1, 76.3), turned to 90 degrees
- moved C2 0.58 mm to (214.3, 46.8)
- moved C1 0.42 mm to (187.1, 35.9)
Connections:
- U1 pad J1_1: (no net) -> +3.3V
- U1 pad J1_10: (no net) -> unconnected-(U1A-GPIO104/I2CSDAA-PadJ1_10)
- U1 pad J1_2: (no net) -> unconnected-(U1A-GPIO32-PadJ1_2)
- U1 pad J1_3: (no net) -> unconnected-(U1A-GPIO19/SCIRXDB-PadJ1_3)
- U1 pad J1_4: (no net) -> unconnected-(U1A-GPIO18/SCITXDB-PadJ1_4)
- U1 pad J1_5: (no net) -> unconnected-(U1A-GPIO67-PadJ1_5)
- U1 pad J1_6: (no net) -> unconnected-(U1A-GPIO111-PadJ1_6)
- U1 pad J1_7: (no net) -> unconnected-(U1A-GPIO60/SPICLKA-PadJ1_7)
- U1 pad J1_8: (no net) -> unconnected-(U1A-GPIO22-PadJ1_8)
- U1 pad J1_9: (no net) -> unconnected-(U1A-GPIO105/I2CSCLA-PadJ1_9)
- U1 pad J3_10: unconnected-(U1C-ADCINA0/ANALOGIN(DACA)-PadJ3_10) -> VHV_S
- U1 pad J3_4: VHV_S -> unconnected-(U1C-ADCINC3/ANALOGIN-PadJ3_4)
- U1 pad J7_1: 5V -> unconnected-(U1G-+5V_J7-PadJ7_1)
- U2 pad 10: (no net) -> +3.3V
- U2 pad 9: 5V -> +3.3V
Routing:
- net 5V: track 138.7 -> 4.65 mm, vias 1 -> 0
- net +3.3V: track 0.00 -> 42.5 mm
- net VHV_S: track 82.0 -> 60.5 mm
- net GND: track 81.8 -> 71.3 mm, vias 16 -> 18
- net Io_S: track 36.7 -> 45.1 mm
- added copper zone on B.Cu, net 5V

Commit message: PCB about done
Parts:
- moved C2 21.2 mm to (214.4, 67.9), turned to -90 degrees
- moved C4 7.75 mm to (166.5, 74.0)
- moved R4 4.46 mm to (126.7, 90.6)
- moved C5 2.53 mm to (113.1, 74.0)
- moved C6 2.53 mm to (110.6, 74.0)
- moved C11 2.14 mm to (149.2, 83.8), turned to 90 degrees
- moved R6 0.07 mm to (128.3, 85.8)
Connections:
- U1 pad J3_10: VHV_S -> unconnected-(U1C-ADCINA0/ANALOGIN(DACA)-PadJ3_10)
- U1 pad J3_8: unconnected-(U1C-ADCINB2/ANALOGIN-PadJ3_8) -> VHV_S
- U1 pad J7_3: Vo_S -> unconnected-(U1G-ADCIN15/ANALOGIN-PadJ7_3)
- U1 pad J7_4: Io_S -> Vo_S
- U1 pad J7_5: unconnected-(U1G-ADCINB5/ANALOGIN-PadJ7_5) -> Io_S
- U2 pad 4: (no net) -> GND
- U2 pad 5: (no net) -> unconnected-(U2-NC-Pad5)
- U2 pad 7: (no net) -> GND
- U2 pad 8: (no net) -> +3.3V
Routing:
- net GND: track 71.3 -> 371.8 mm, vias 18 -> 20
- net VHV_S: track 60.5 -> 67.2 mm
- net Vo_S: track 21.7 -> 26.6 mm
- net 5V: track 4.65 -> 0.00 mm
- net Io_S: track 45.1 -> 49.1 mm
- net Vo: track 2.80 -> 0.00 mm
- net +3.3V: track 42.5 -> 43.9 mm
- net Net-(R5-Pad1): track 2.86 -> 3.45 mm

Commit message: PCB complete
Connections:
- net Net-(U2-IN+) renamed /Voh
Routing:
- net GND: track 371.8 -> 372.8 mm
- net VHV_S: track 67.2 -> 68.0 mm

Commit message: PCB ORDERED
This push contains the PCB version and Gerber files that were ordered for the first prototype.
Parts:
- moved J5 1.50 mm to (188.0, 140.8)
- moved C1 0.27 mm to (187.0, 35.6)
- moved C8 0.18 mm to (120.8, 132.5)
Connections:
- C2 pad 1: 5V -> +3.3V
- J1 pad 3: 5V -> +3.3V
- J2 pad 1: 5V -> +3.3V
Routing:
- net GND: track 372.8 -> 56.7 mm, vias 20 -> 19
- added copper zone on B.Cu, net +3.3V
- removed copper zone on B.Cu, net 5V
