File: Battery Charger Project/KiCad/Wind charger/Wind charger.kicad_sch (KiCad schematic)
At the start: 11 parts, among them Q1 NMOS, U1 TMCS1133C3A

Commit message: started on schematic
Parts:
- U2: value ~ -> (none)

Commit message: Added demo folder
Parts:
- removed R1: 15kΩ, symbol Device:R
- removed R2: 1.8kΩ, symbol Device:R
- added R4, R5, R6, R7: R_US, symbol Device:R_US
Connections:
- net +3.3V is gone; now on net +5V: U1.9 (VS)
- net GND: now also R5.2, R7.2
- net HV: now also R6.1
- net at BT1.1 (+), U1.2 (IN-): now also R4.1
- net AI1 renamed Io_S
- new net VHV_S: R6.2, R7.1
- new net Vo_S: R4.2, R5.1

Commit message: Made presentation and added footprintst
I finished the presentation. This required me to remove some things from the simulation to make it more understandable. I also just about finished adding all the footprints for the PCB
Parts:
- C1: value 7.15μF -> 10μF
- C2: value 1μF -> 2.2mF
- L1: renamed from 6.51µF; value 6.51µH -> 437µH
- U1: value TMCS1133C3A -> TMCS1133C5A
Other:
- note added: ": CONNECTION ON EVAL BOARD"
- note removed: "= CONNECTION ON EVAL BOARD"
